Commit message: ..

File: src/warthog_description/urdf/warthog.urdf.xacro (robot description, xacro)
@@ -448,4 +448,10 @@
     <child link="imu_link" />
   </joint>
+  <link name="gps_link"/>
+  <joint name="gps_link_joint" type="fixed">
+    <parent link="chassis_link"/>
+    <child link="gps_link"/>
+    <origin xyz="0 0 0" rpy="0 0 0"/>
+  </joint>
   <!-- Bring in simulation data for Gazebo. -->
   <xacro:include filename="$(find warthog_description)/urdf/warthog.gazebo" />

Commit message: test nhung ma loi

File: src/warthog_description/urdf/warthog.urdf.xacro (robot description, xacro)
@@ -438,5 +438,5 @@
   </link>
   <joint name="diff_link_joint" type="fixed">
-    <parent link="chassis_link"/>
+    <parent link="base_link"/>
     <child link="diff_link"/>
     <origin xyz="-0.5826 0 0.24979" rpy="0 0 0" />
@@ -450,5 +450,5 @@
   <link name="gps_link"/>
   <joint name="gps_link_joint" type="fixed">
-    <parent link="chassis_link"/>
+    <parent link="base_link"/>
     <child link="gps_link"/>
     <origin xyz="0 0 0" rpy="0 0 0"/>

Commit message: add_outdoor_waypoint_nav

File: src/warthog_description/urdf/warthog.urdf.xacro (robot description, xacro)
@@ -454,4 +454,10 @@
     <origin xyz="0 0 0" rpy="0 0 0"/>
   </joint>
+  <link name="front_laser"/>
+  <joint name="front_laser_joint" type="fixed">
+    <parent link="base_link"/>
+    <child link="front_laser"/>
+    <origin xyz="0 0 0" rpy="0 0 0"/>
+  </joint>
   <!-- Bring in simulation data for Gazebo. -->
   <xacro:include filename="$(find warthog_description)/urdf/warthog.gazebo" />

Commit message: như_branch

File: src/warthog_description/urdf/warthog.urdf.xacro (robot description, xacro)
@@ -456,7 +456,7 @@
   <link name="front_laser"/>
   <joint name="front_laser_joint" type="fixed">
-    <parent link="base_link"/>
+    <parent link="top_chassis_link"/>
     <child link="front_laser"/>
-    <origin xyz="0 0 0" rpy="0 0 0"/>
+    <origin xyz="0.4 0 0.549" rpy="0 0 0"/>
   </joint>
   <!-- Bring in simulation data for Gazebo. -->
