Commit message: update_send_data

File: src/warthog_navigation/warthog_simulation/urdf/sick_lms1xx_mount.urdf.xacro (robot description, xacro)
@@ -27,6 +27,6 @@
 <robot xmlns:xacro="http://www.ros.org/wiki/xacro">
   <xacro:include filename="$(find lms1xx)/urdf/sick_lms1xx.urdf.xacro" />
-  <xacro:macro name="sick_lms1xx_mount" params="prefix topic parent_link *origin">
-    <xacro:sick_lms1xx frame="${prefix}_laser" topic="${topic}" />
+  <xacro:macro name="sick_lms1xx_mount" params="prefix topic parent_link max_range:=100.0 *origin">
+    <xacro:sick_lms1xx frame="${prefix}_laser" topic="${topic}" max_range="${max_range}" />
     <joint name="${prefix}_laser_mount_joint" type="fixed">
       <xacro:insert_block name="origin" />

File: src/warthog_navigation/warthog_simulation/urdf/warthog_nav.urdf.xacro (robot description, xacro)
@@ -10,12 +10,5 @@
     <origin xyz="0.4 0.0 0.4" rpy="0 0 0" />
   </xacro:VLP-16> -->
-  <!-- LMS1xx Laser Scan -->
-  <xacro:include filename="$(find warthog_simulation)/urdf/sick_lms1xx_mount.urdf.xacro" />
-  <xacro:sick_lms1xx_mount prefix="front"
-        parent_link="top_chassis_link"
-        topic="front/scan">
-    <origin xyz="0.4 0.0 0.4"
-            rpy="0 0 0" />
-  </xacro:sick_lms1xx_mount>
+  <!-- /front/scan is provided by warthog_description/urdf/warthog.gazebo. -->
   <!-- Realsense D435 -->
   <xacro:include filename="$(find warthog_simulation)/urdf/realsense.urdf.xacro"/>
